File: PCBs/DDI-parent/DDI-parent.kicad_pcb (KiCad board)
At the start: 2 copper layers, 101 x 12.5 mm, 27 parts, among them J1 VCC, J10 GND, J11 SCL, J12 SDA, J13 IRQ, J14 VCC, J15 GND, J2 GND, J3 SCL, J4 SDA, J5 IRQ, J6 SCL, J7 SDA, J8 IRQ, J9 VCC, SW1 TL1240GQ, SW2 TL1240GQ, SW3 TL1240GQ, SW4 TL1240GQ, SW5 TL1240GQ, U1 TCA9554PWR

Commit message: new stuff
Parts:
- added J16: RGND, Connector_Wire:SolderWirePad_1x01_SMD_4x3mm, F.Cu at (201.0, -214.9)
- added J17: RA, Connector_Wire:SolderWirePad_1x01_SMD_4x3mm, F.Cu at (197.5, -214.9)
- added J18: RB, Connector_Wire:SolderWirePad_1x01_SMD_4x3mm, F.Cu at (194.0, -214.9)
- C1: value 1uF -> 47uf; footprint Capacitor_THT:CP_Radial_D3.0mm_P5.00mm -> Capacitor_SMD:C_1206_3216Metric
- J10, J11: footprint Connector_PinHeader_1.00mm:PinHeader_1x01_P1.00mm_Vertical -> Connector_Wire:SolderWirePad_1x01_SMD_4x3mm; moved to F.Cu
- J7, J8, J9: footprint Connector_PinHeader_1.00mm:PinHeader_1x01_P1.00mm_Vertical -> Connector_Wire:SolderWirePad_1x01_SMD_4x3mm
- moved J9 103.2 mm to (156.8, -208.4), turned to -90 degrees
- moved J8 100.0 mm to (156.9, -211.9)
- moved J11 99.7 mm to (160.4, -214.2), turned to -135 degrees
- moved J10 97.9 mm to (156.8, -208.4), turned to 90 degrees
- moved J7 96.6 mm to (160.4, -214.2), turned to -135 degrees
- moved A2 37.9 mm to (166.8, -212.8)
- moved J3 23.9 mm to (200.9, -214.9)
- moved J1 21.3 mm to (195.2, -209.0)
- moved A1 20.7 mm to (179.6, -208.0)
- moved J2 20.5 mm to (194.0, -214.4)
- moved J4 20.4 mm to (199.8, -208.9)
- moved U1 20.3 mm to (177.8, -213.4)
- moved J5 16.9 mm to (197.5, -214.9)
- moved A0 12.8 mm to (174.6, -208.0), turned to 0 degrees
- moved C1 4.21 mm to (173.6, -213.5), turned to -90 degrees
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Connections:
- U1 pad 10: unconnected-(U1-P5-Pad10) -> /U1P5
- U1 pad 11: unconnected-(U1-P6-Pad11) -> /U1P6
Routing:
- net GND: track 96.7 -> 166.2 mm, vias 3 -> 5
- net /U1P3: track 0.00 -> 53.9 mm
- net IRQ: track 97.7 -> 56.8 mm, vias 3 -> 4
- net +5V: track 129.3 -> 89.4 mm, vias 10 -> 7
- net /U1P2: track 6.44 -> 42.2 mm, vias 0 -> 1
- net /U1P4: track 58.2 -> 84.1 mm, vias 0 -> 2
- net /U1P0: track 32.7 -> 7.97 mm
- net /U1P6: track 0.00 -> 20.7 mm
- net SCL: track 100.6 -> 120.4 mm, vias 3 -> 6
- net SDA: track 90.9 -> 102.5 mm
- net /A1: track 8.35 -> 0.00 mm, vias 1 -> 0
- net /A0: track 9.53 -> 3.37 mm
- net /A2: track 11.4 -> 14.3 mm
Other:
- board size 101 x 12.5 mm -> 102 x 11.7 mm
- board text added: "Erik Goldman, 2024"
- board text removed: "1uF"

Commit message: shipped off v1.1
Parts:
- C1: value 47uf -> 0.1uF; footprint Capacitor_SMD:C_1206_3216Metric -> Capacitor_SMD:C_0402_1005Metric
Routing:
- net IRQ: track 56.8 -> 98.3 mm, vias 4 -> 5
- net +5V: track 89.4 -> 114.4 mm
- net /U1P5: track 0.00 -> 21.1 mm
- net /U1P0: track 7.97 -> 18.5 mm, vias 0 -> 3
- net GND: track 166.2 -> 158.3 mm
- net /U1P1: track 10.7 -> 18.5 mm
- net /U1P3: track 53.9 -> 61.2 mm
- net /A1: track 0.00 -> 6.20 mm, vias 0 -> 1
- net /U1P6: track 20.7 -> 17.9 mm
- net /A2: track 14.3 -> 12.6 mm, vias 1 -> 3
- net /U1P4: track 84.1 -> 85.1 mm
Other:
- board text added: "DDI v1.1"
- board text removed: "DDI v1"

Commit message: stash
Parts:
- SW1, SW2, SW3, SW4, SW5: footprint OH_Footprints:TL1240GQ -> Library:TL1240GQ
Routing:
- net SCL: track 120.3 -> 115.3 mm
- net +5V: track 114.4 -> 110.7 mm
- net IRQ: track 98.3 -> 94.8 mm
- net SDA: track 102.1 -> 100.7 mm
- net /A1: track 6.20 -> 7.56 mm
- net /A0: track 3.37 -> 4.37 mm
