File: PCBs/DDI-parent/DDI-parent.kicad_sch (KiCad schematic)
At the start: 25 parts, among them J1 VCC, J10 GND, J11 SCL, J12 SDA, J13 IRQ, J14 VCC, J15 GND, J2 GND, J3 SCL, J4 SDA, J5 IRQ, J6 SCL, J7 SDA, J8 IRQ, J9 VCC, SW1 TL1240GQ, SW2 TL1240GQ, SW3 TL1240GQ, SW4 TL1240GQ, SW5 TL1240GQ, U1 TCA9554PWR

Commit message: new stuff
Parts:
- added J16: RGND, Connector_Wire:SolderWirePad_1x01_SMD_4x3mm, symbol Connector:Conn_01x01_Pin
- added J17: RA, Connector_Wire:SolderWirePad_1x01_SMD_4x3mm, symbol Connector:Conn_01x01_Pin
- added J18: RB, Connector_Wire:SolderWirePad_1x01_SMD_4x3mm, symbol Connector:Conn_01x01_Pin
- C1: value 1uF -> 47uf; footprint Capacitor_THT:CP_Radial_D3.0mm_P5.00mm -> Capacitor_SMD:C_1206_3216Metric
- J10, J11, J7, J8, J9: footprint Connector_PinHeader_1.00mm:PinHeader_1x01_P1.00mm_Vertical -> Connector_Wire:SolderWirePad_1x01_SMD_4x3mm
- renumbered JP1 to A0, JP2 to A1, JP3 to A2
Connections:
- net GND: now also J16.1 (Pin_1)
- net U1P5: now reaches U1.10 (P5)
- net U1P5: now also J17.1 (Pin_1)
- net U1P6: now reaches U1.11 (P6)
- net U1P6: now also J18.1 (Pin_1)
- no-connect marks 3 -> 1

Commit message: shipped off v1.1
Parts:
- C1: value 47uf -> 0.1uF; footprint Capacitor_SMD:C_1206_3216Metric -> Capacitor_SMD:C_0402_1005Metric
Changed lines of the file:
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@@
 			)
 		)
-		(property "Value" "47uf"
+		(property "Value" "0.1uF"
 			(at 95.25 49.53 0)
 			(effects
@@
 			)
 		)
-		(property "Footprint" "Capacitor_SMD:C_1206_3216Metric"
+		(property "Footprint" "Capacitor_SMD:C_0402_1005Metric"
 			(at 93.6752 52.07 0)
 			(effects

Commit message: stash
Parts:
- SW1, SW2, SW3, SW4, SW5: footprint KiCAD Libraries:TL1240GQ -> Library:TL1240GQ
Changed lines of the file:
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@@
 			)
 		)
-		(property "Footprint" "KiCAD Libraries:TL1240GQ"
+		(property "Footprint" "Library:TL1240GQ"
 			(at 67.056 73.152 0)
 			(effects
@@
 			)
 		)
-		(property "Footprint" "KiCAD Libraries:TL1240GQ"
+		(property "Footprint" "Library:TL1240GQ"
 			(at 91.186 73.152 0)
 			(effects
@@
 			)
 		)
-		(property "Footprint" "KiCAD Libraries:TL1240GQ"
+		(property "Footprint" "Library:TL1240GQ"
 			(at 115.316 73.152 0)
 			(effects
@@
 			)
 		)
-		(property "Footprint" "KiCAD Libraries:TL1240GQ"
+		(property "Footprint" "Library:TL1240GQ"
 			(at 67.056 87.122 0)
 			(effects
@@
 			)
 		)
-		(property "Footprint" "KiCAD Libraries:TL1240GQ"
+		(property "Footprint" "Library:TL1240GQ"
 			(at 91.186 87.122 0)
 			(effects
